File: leddriver.sch (KiCad schematic (older format))
At the start: 46 parts, among them U1 LNK3202/3204-6

Commit message: Finished Schematic
Parts:
- removed C? (x4): C, symbol C
- removed R?: R, symbol R
- added C10, C9: 18p, Capacitors_SMD:C_0805_HandSoldering, symbol C
- added C17, C18: 22p, Capacitors_SMD:C_0805_HandSoldering, symbol C
- added D4, D6, D7: LED, LEDs:LED_D5.0mm, symbol LED
- added J3, J5: CONN_02X03, Pin_Headers:Pin_Header_Straight_2x03_Pitch2.54mm, symbol CONN_02X03
- added J4: USB_OTG, Connectors:USB_Micro-B_10103594-0001LF, symbol USB_OTG
- added Q2, Q3: S8050, TO_SOT_Packages_THT:TO-92_Molded_Narrow, symbol S8050
- added R10, R25, R8: 1k, Resistors_SMD:R_0805_HandSoldering, symbol R
- added R12, R13, R14, R15, R18: 10k, Resistors_SMD:R_0805_HandSoldering, symbol R
- added R16, R17: 12k, Resistors_SMD:R_0805_HandSoldering, symbol R
- added R23, R24: 470, Resistors_SMD:R_0805_HandSoldering, symbol R
- added R26, R4: 0.009, Resistors_SMD:R_2512_HandSoldering, symbol R
- added RV2: 10k, Potentiometers:Potentiometer_Trimmer_Bourns_3299Y, symbol POT
- added U5: esp8266mod, symbol esp8266mod
- added U6: CH340G, SMD_Packages:SO-16-N, symbol CH340G
- added Y1: 16MHz, Crystals:Crystal_SMD_HC49-SD_HandSoldering, symbol Crystal
- added Y2: Crystal, Crystals:Crystal_SMD_HC49-SD_HandSoldering, symbol Crystal
- C1: footprint (none) -> Capacitors_SMD:C_0805_HandSoldering
- C12: renamed from C?; value C -> 0.068uF; footprint (none) -> Capacitors_SMD:C_1812_HandSoldering
- C14: renamed from C?; value C -> 1000uF; footprint (none) -> Capacitors_THT:CP_Radial_D35.0mm_P10.00mm_SnapIn
- C15, C16: renamed from C?; footprint (none) -> Capacitors_SMD:C_0805_HandSoldering
- C2: footprint (none) -> Capacitors_SMD:CP_Elec_4x5.3
- C5: renamed from C?; value C -> 10n; footprint (none) -> Capacitors_SMD:C_1206_HandSoldering
- C7: renamed from C?; value C -> 2.2u; footprint (none) -> Capacitors_SMD:CP_Elec_4x5.3
- C8: footprint (none) -> Capacitors_SMD:CP_Elec_6.3x5.3
- D1, D3: footprint (none) -> TO_SOT_Packages_SMD:TO-252-2Lead
- D2: renamed from D?; footprint (none) -> TO_SOT_Packages_SMD:TO-252-2Lead
- DS1: renamed from DS?; footprint RC1602A -> Pin_Headers:Pin_Header_Straight_1x16_Pitch2.54mm
- F1: renamed from F?; footprint (none) -> Fuse_Holders_and_Fuses:Fuseholder5x20_horiz_open_inline_Type-I
- J2: renamed from J?; footprint (none) -> Connectors_Phoenix:PhoenixContact_MSTB-GF_02x5.08mm_Angled_ThreadedFlange
- J6: renamed from J?; footprint (none) -> Pin_Headers:Pin_Header_Straight_1x04_Pitch2.54mm
- L1: footprint (none) -> Choke_SMD:Choke_SMD_7.3x7.3_H4.5
- L2: renamed from L?; footprint (none) -> Inductors_THT:L_Toroid_Vertical_L25.4mm_W14.7mm_P12.20mm_Vishay_TJ5
- Q1: renamed from Q?; footprint (none) -> TO_SOT_Packages_SMD:TO-252-2Lead
- R1, R2, R3, R5: footprint (none) -> Resistors_SMD:R_0805_HandSoldering
- R11: renamed from R?; value R -> 0.15; footprint (none) -> Resistors_THT:R_Axial_DIN0414_L11.9mm_D4.5mm_P15.24mm_Horizontal
- R19, R20, R21, R22, R9: renamed from R?; footprint (none) -> Resistors_SMD:R_0805_HandSoldering
- R6: renamed from R?; value R -> 300k; footprint (none) -> Resistors_SMD:R_0805_HandSoldering
- R7: renamed from R?; value R -> 1k; footprint (none) -> Resistors_SMD:R_0805_HandSoldering
- RV1: renamed from RV?; footprint (none) -> Varistors:RV_Disc_D7_W4.8_P5
- U1: footprint (none) -> SMD_Packages:SOIC-8-N
- U3: renamed from U?; footprint (none) -> SMD_Packages:SOIC-8-N
- gave numbers to parts that had none: 7
Connections:
- net +3V3: now also DS1.1 (VSS), DS1.15 (LED+), U2.18 (AVCC), U2.20 (AREF), U2.4 (VCC), U2.6 (VCC), J3.2 (P2), R12.2, R13.2, R14.1, R18.1, RV2.1, U5.8 (Vcc), U6.16 (VCC), U6.4 (V3)
- net Enc_A: now also U2.24 ((PCINT9/ADC1)PC1)
- net Enc_B: now also U2.25 ((PCINT10/ADC2)PC2)
- net GND: now also DS1.16 (LED-), DS1.2 (VDD), U2.21 (GND), U2.3 (GND), U2.5 (GND), C10.2, C17.1, C18.1, C9.2, D4.1 (K), D6.1 (K), D7.1 (K), J3.6 (P6), J4.5 (GND), J4.6 (Shield), R15.1, R4.1, RV2.3, U5.15 (GND), U6.1 (GND)
- net Knob_A: now also U2.32 ((PCINT18/INT0)PD2)
- net Knob_B: now also U2.1 ((PCINT19/OC2B/INT1)PD3)
- net Knob_SW: now also U2.12 ((PCINT0/CLKO/ICP1)PB0)
- net PWM: now also U2.13 ((PCINT1/OC1A)PB1), R10.2
- net at Q1.3 (S), U3.2 (CS): now also R26.1
- net D6: now reaches U2.10 ((PCINT22/OC0A/AIN0)PD6)
- net D6: now also DS1.13 (DB6)
- net D7: now reaches U2.11 ((PCINT23/AIN1)PD7)
- net D7: now also DS1.14 (DB7)
- net at U2.14 ((PCINT2/OC1B/~SS~)PB2): now also R8.2
- net at U2.15 ((PCINT3/OC2A/MOSI)PB3): now also J3.4 (P4)
- net at U2.16 ((PCINT4/MISO)PB4): now also DS1.4 (RS), J3.1 (P1)
- net at U2.17 ((PCINT5/SCK)PB5): now also DS1.5 (R/~W), J3.3 (P3)
- net D4: now reaches U2.2 ((PCINT20/XCK/T0)PD4)
- net D4: now also DS1.11 (DB4)
- net at U2.23 ((PCINT8/ADC0)PC0): now also DS1.6 (E)
- net IC_CLK: now reaches U2.26 ((PCINT11/ADC3)PC3)
- net IC_CLK: now also U5.20 (IO_5)
- net IC_DAT: now reaches U2.27 ((PCINT12/SDA/ADC4)PC4)
- net IC_DAT: now also U5.19 (IO_4)
- net IC_AUX: now reaches U2.28 ((PCINT13/SCL/ADC5)PC5)
- net IC_AUX: now also U5.4 (IO_16)
- net RST: now reaches U2.29 ((PCINT14/~RESET~)PC6)
- net RST: now also J3.5 (P5), Q2.3 (C), R12.1, U5.1 (/RST)
- net AVR_RX: now reaches U2.30 ((PCINT16/RXD)PD0)
- net AVR_RX: now also J5.1 (P1)
- net AVR_TX: now reaches U2.31 ((PCINT17/TXD)PD1)
- net AVR_TX: now also J5.2 (P2)
- net at U2.7 ((PCINT6/XTAL1/TOSC1)PB6): now also C10.1, Y1.1
- net at U2.8 ((PCINT7/XTAL2/TOSC2)PB7): now also C9.1, Y1.2
- net D5: now reaches U2.9 ((PCINT21/OC0B/T1)PD5)
- net D5: now also DS1.12 (DB5)
- net at DS1.3 (Vo): now also RV2.2
- new net: R15.2, U5.16 (IO_15)
- new net: R14.2, U5.17 (IO_2)
- new net: R13.1, U5.3 (EN)
- new net: R25.1, U5.5 (IO_14)
- new net: Q2.1 (E), R17.1, U6.14 (/RTS)
- new net: Q2.2 (B), R16.2
- new net: Q3.1 (E), R16.1, U6.13 (/DTR)
- new net: Q3.2 (B), R17.2
- new net: R23.2, U6.3 (RXD)
- new net: R24.2, U6.2 (TXD)
- new net: C18.2, U6.7 (XI), Y2.2
- new net: C17.2, U6.8 (XO), Y2.1
- new net: D4.2 (A), R8.1
- new net: D6.2 (A), R10.1
- new net: D7.2 (A), R25.2
- new net: R26.2, R4.2
- new net ESP_RX: J5.5 (P5), U5.21 (RXD)
- new net ESP_TX: J5.6 (P6), U5.22 (TXD)
- new net GPIO0: Q3.3 (C), R18.2, U5.18 (IO_0)
- new net RXD: J5.3 (P3), R24.1
- new net TXD: J5.4 (P4), R23.1
- new net USB+: J4.3 (D+), U6.5 (UD+)
- new net USB-: J4.2 (D-), U6.6 (UD-)
- no-connect marks 0 -> 22
Other:
- note added: "400W LED Strobe Driver"
- moved on the sheet: C1, C15, C16, C2, C8, D1, D3, DS1, J2, J6, L1, R1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

Commit message: PCB
Parts:
- removed D1, D2, D3: D, TO_SOT_Packages_SMD:TO-252-2Lead, symbol D
- added D1, D2, D3: ThreepinDiode, TO_SOT_Packages_SMD:TO-252-2_Rectifier, symbol ThreepinDiode
- C3: footprint (none) -> local_footprints:703w-00-53
- D5: footprint (none) -> local_footprints:ds21221
- J1: footprint (none) -> Connectors:1pin
- L3: footprint (none) -> local_footprints:pm3700
- Q1: footprint TO_SOT_Packages_SMD:TO-252-2Lead -> TO_SOT_Packages_SMD:TO-252-2
- SW1: footprint (none) -> local_footprints:pec12r
- U2: footprint TQFP32 -> Housings_QFP:TQFP-32_7x7mm_Pitch0.8mm
- U5: footprint (none) -> local_footprints:ESP12E
Connections:
- net +3V3: now also D2.3
- net GND: now also D3.3
- net HT: now also D1.2
- net at J1.1 (P1), L2.2, Q1.2 (D): now also D1.3
- net at C1.1, C2.2, L1.1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: now also D3.2
- net at C2.1, R1.1, R3.2: now also D2.2
Changed lines of the file:
@@
 F 0 "C3" H 1100 1250 60  0000 C CNN
 F 1 "703w-00/53" H 1100 1350 60  0000 C CNN
-F 2 "" H 1100 1100 60  0001 C CNN
+F 2 "local_footprints:703w-00-53" H 1100 1100 60  0001 C CNN
 F 3 "" H 1100 1100 60  0001 C CNN
 	1    1100 1100
@@
 F 0 "L3" H 2850 950 60  0000 C CNN
 F 1 "CHOKE" H 2850 1350 60  0000 C CNN
-F 2 "" H 2950 1300 60  0001 C CNN
+F 2 "local_footprints:pm3700" H 2950 1300 60  0001 C CNN
 F 3 "" H 2950 1300 60  0001 C CNN
 	1    2850 1150
@@
 F 0 "D5" H 3750 1425 50  0000 L CNN
 F 1 "D_Bridge_+AA-" H 3750 1350 50  0000 L CNN
-F 2 "" H 3700 1150 50  0001 C CNN
+F 2 "local_footprints:ds21221" H 3700 1150 50  0001 C CNN
 F 3 "" H 3700 1150 50  0001 C CNN
 	1    3700 1150
@@
 F 0 "Q1" H 1350 1950 50  0000 L CNN
 F 1 "Q_NMOS_GDS" V 1550 2000 50  0000 L CNN
-F 2 "TO_SOT_Packages_SMD:TO-252-2Lead" H 1550 2300 50  0001 C CNN
+F 2 "TO_SOT_Packages_SMD:TO-252-2" H 1550 2300 50  0001 C CNN
 F 3 "" H 1350 2200 50  0001 C CNN
 	1    1350 2200
@@
 $EndComp
 $Comp
-L D D2
-U 1 1 5930FC0A
-P 1050 2750
-F 0 "D2" H 1050 2850 50  0000 C CNN
-F 1 "D" H 1050 2650 50  0000 C CNN
-F 2 "TO_SOT_Packages_SMD:TO-252-2Lead" H 1050 2750 50  0001 C CNN
-F 3 "" H 1050 2750 50  0001 C CNN
-	1    1050 2750
-	1    0    0    -1
-$EndComp
-$Comp
 L C C7
 U 1 1 5930FCC5
@@
 F 0 "U2" H 1150 7100 50  0000 L BNN
 F 1 "ATMEGA328P-AU" H 2300 4450 50  0000 L BNN
-F 2 "TQFP32" H 1900 5850 50  0001 C CIN
+F 2 "Housings_QFP:TQFP-32_7x7mm_Pitch0.8mm" H 1900 5850 50  0001 C CIN
 F 3 "" H 1900 5850 50  0001 C CNN
 	1    1900 5850
@@
 F 0 "J1" H 1500 2550 50  0000 C CNN
 F 1 "CONN_01X01" V 1600 2450 50  0000 C CNN
-F 2 "" H 1500 2450 50  0001 C CNN
+F 2 "Connectors:1pin" H 1500 2450 50  0001 C CNN
 F 3 "" H 1500 2450 50  0001 C CNN
 	1    1500 2450
@@
 L HT #PWR03
 U 1 1 59310FDA
-P 900 2750
-F 0 "#PWR03" H 900 2870 50  0001 C CNN
-F 1 "HT" H 900 2840 50  0000 C CNN
-F 2 "" H 900 2750 50  0001 C CNN
-F 3 "" H 900 2750 50  0001 C CNN
-	1    900  2750
-	1    0    0    -1
+P 1200 3200
+F 0 "#PWR03" H 1200 3320 50  0001 C CNN
+F 1 "HT" H 1200 3290 50  0000 C CNN
+F 2 "" H 1200 3200 50  0001 C CNN
+F 3 "" H 1200 3200 50  0001 C CNN
+	1    1200 3200
+	-1   0    0    1
 $EndComp
 $Comp
@@
 $EndComp
 $Comp
-L D D1
-U 1 1 5931592F
-P 8950 900
-F 0 "D1" H 8950 1000 50  0000 C CNN
-F 1 "D" H 8950 800 50  0000 C CNN
-F 2 "TO_SOT_Packages_SMD:TO-252-2Lead" H 8950 900 50  0001 C CNN
-F 3 "" H 8950 900 50  0001 C CNN
-	1    8950 900
-	0    1    1    0
-$EndComp
-$Comp
 L L L1
 U 1 1 59315984
@@
 $EndComp
 $Comp
-L D D3
-U 1 1 593159E9
-P 9900 1700
-F 0 "D3" H 9900 1800 50  0000 C CNN
-F 1 "D" H 9900 1600 50  0000 C CNN
-F 2 "TO_SOT_Packages_SMD:TO-252-2Lead" H 9900 1700 50  0001 C CNN
-F 3 "" H 9900 1700 50  0001 C CNN
-	1    9900 1700
-	0    1    1    0
-$EndComp
-$Comp
 L HT #PWR014
 U 1 1 59318272
@@
 L GND #PWR015
 U 1 1 593254F8
-P 9900 1850
-F 0 "#PWR015" H 9900 1600 50  0001 C CNN
-F 1 "GND" H 9900 1700 50  0000 C CNN
-F 2 "" H 9900 1850 50  0001 C CNN
-F 3 "" H 9900 1850 50  0001 C CNN
-	1    9900 1850
+P 9900 2000
+F 0 "#PWR015" H 9900 1750 50  0001 C CNN
+F 1 "GND" H 9900 1850 50  0000 C CNN
+F 2 "" H 9900 2000 50  0001 C CNN
+F 3 "" H 9900 2000 50  0001 C CNN
+	1    9900 2000
 	1    0    0    -1
 $EndComp
@@
 F 0 "SW1" H 10300 5210 50  0000 C CNN
 F 1 "Rotary_Encoder_Switch" H 10500 4700 50  0000 C CNN
-F 2 "" H 10200 5110 50  0001 C CNN
+F 2 "local_footprints:pec12r" H 10200 5110 50  0001 C CNN
 F 3 "" H 10300 5210 50  0001 C CNN
 	1    10300 4950
@@
 F 0 "U5" H 5050 6900 60  0000 C CNN
 F 1 "esp8266mod" H 5100 7300 60  0000 C CNN
-F 2 "" H 5050 5900 60  0001 C CNN
+F 2 "local_footprints:ESP12E" H 5050 5900 60  0001 C CNN
 F 3 "" H 5050 5900 60  0001 C CNN
 	1    5050 6900
@@
 	10850 700  10250 700
 Wire Wire Line
-	9650 700  8950 700
-Wire Wire Line
-	8950 700  8950 750
-Wire Wire Line
 	9600 750  9600 700
 Connection ~ 9600 700
 Wire Wire Line
-	9300 950  9300 700
+	9300 600  9300 950
 Connection ~ 9300 700
 Wire Wire Line
@@
 Wire Wire Line
 	800  1950 800  2000
+$Comp
+L ThreepinDiode D1
+U 1 1 593216F7
+P 1350 3000
+F 0 "D1" H 1350 3000 60  0000 C CNN
+F 1 "ThreepinDiode" H 1350 3300 60  0000 C CNN
+F 2 "TO_SOT_Packages_SMD:TO-252-2_Rectifier" H 1350 3000 60  0001 C CNN
+F 3 "" H 1350 3000 60  0001 C CNN
+	1    1350 3000
+	0    -1   -1   0
+$EndComp
+$Comp
+L ThreepinDiode D3
+U 1 1 5932423A
+P 9750 1750
+F 0 "D3" H 9750 1750 60  0000 C CNN
+F 1 "ThreepinDiode" H 9750 2050 60  0000 C CNN
+F 2 "TO_SOT_Packages_SMD:TO-252-2_Rectifier" H 9750 1750 60  0001 C CNN
+F 3 "" H 9750 1750 60  0001 C CNN
+	1    9750 1750
+	0    1    1    0
+$EndComp
+$Comp
+L ThreepinDiode D2
+U 1 1 59324B9B
+P 8800 800
+F 0 "D2" H 8800 800 60  0000 C CNN
+F 1 "ThreepinDiode" H 8800 1100 60  0000 C CNN
+F 2 "TO_SOT_Packages_SMD:TO-252-2_Rectifier" H 8800 800 60  0001 C CNN
+F 3 "" H 8800 800 60  0001 C CNN
+	1    8800 800
+	0    1    1    0
+$EndComp
+Wire Wire Line
+	8950 600  9300 600
+Wire Wire Line
+	9300 700  9650 700
 $EndSCHEMATC
